File: kicad/ggsmdriver.kicad_pcb (KiCad board)
At the start: 4 copper layers, 55 x 45 mm, 65 parts, among them J3 VIN GND A2 A1 B1 B2, J4 EXP, J5 USB-C, SW1 BOOT, SW2 RESET, U1 STM32G0B1CBT6, U2 TMC2209-LA-T, U3 TPS54202DDCR, U4 XC6206P332MR, U5 USBLC6-2SC6

Commit message: Add STDC14 debug connector for the STLINK-V3MINIE
J6 (Samtec FTSH-107-01-L-DV-K, hand-soldered) on the left under the LEDs:
SWD, NRST, 3V3 sense, GND, and the probe's virtual COM on USART1 (PB6/PB7).
SWD test pads removed. 0 unrouted, DRC clean; fab regenerated.

Co-Authored-By: Claude Opus 5.5 (1M context) <noreply@anthropic.com>
Claude-Session: https://claude.ai/code/session_01VFhb1Qv7mkaGrgvtw2CS4q
Parts:
- removed TP1: +3V3, TestPoint:TestPoint_Pad_D1.0mm
- removed TP2: SWDIO, TestPoint:TestPoint_Pad_D1.0mm
- removed TP3: BOOT0_SWCLK, TestPoint:TestPoint_Pad_D1.0mm
- removed TP4: NRST, TestPoint:TestPoint_Pad_D1.0mm
- removed TP5: GND, TestPoint:TestPoint_Pad_D1.0mm
- added J6: STDC14, Connector_PinHeader_1.27mm:PinHeader_2x07_P1.27mm_Vertical_SMD, F.Cu at (104.5, 124.5)
- moved D1 3.20 mm to (118.5, 135.0)
- moved SW1 0.50 mm to (113.0, 124.5)
- moved SW2 0.50 mm to (113.0, 140.5)
Connections:
- U1 pad 45: (no net) -> VCP_TX
- U1 pad 46: (no net) -> VCP_RX
Routing:
- net VCP_RX: track 0.00 -> 34.2 mm, vias 0 -> 2
- net TMC_UART: track 55.7 -> 23.5 mm, vias 6 -> 3
- net VCP_TX: track 0.00 -> 31.0 mm
- net TMC_DIR: track 56.9 -> 82.1 mm, vias 2 -> 3
- net IO1: track 48.0 -> 29.4 mm
- net ENC_B: track 33.3 -> 46.5 mm
- net NRST: track 24.7 -> 34.7 mm
- net SWDIO: track 36.7 -> 26.7 mm, vias 2 -> 0
- net +3V3: track 153.7 -> 145.0 mm
- net BOOT0_SWCLK: track 42.9 -> 34.4 mm
- net TMC_STEP: track 67.9 -> 74.9 mm, vias 3 -> 4
- net LED_STAT_R: track 45.5 -> 41.2 mm
- net GND: track 71.2 -> 75.5 mm, vias 51 -> 53
- net TMC_EN: track 37.7 -> 34.1 mm
- net TMC_TX: track 19.2 -> 16.2 mm
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