File: kicad/ggsmdriver.kicad_sch (KiCad schematic)
At the start: 65 parts, among them J3 VIN GND A2 A1 B1 B2, J4 EXP, J5 USB-C, SW1 BOOT, SW2 RESET, U1 STM32G0B1CBT6, U2 TMC2209-LA-T, U3 TPS54202DDCR, U4 XC6206P332MR, U5 USBLC6-2SC6

Commit message: Swap Extended passives to JLC Basic, hand-solder the header
C16 -> C21122, C17-19/C23 220nF -> 100nF C14663, C4 75pF -> 100pF C14858.
J4 drops its LCSC number so it stays out of the JLC BOM/CPL. Board
re-routed (0 unrouted, no DRC errors) and fab files regenerated.

Co-Authored-By: Claude Opus 5.5 (1M context) <noreply@anthropic.com>
Claude-Session: https://claude.ai/code/session_01VFhb1Qv7mkaGrgvtw2CS4q
Parts:
- C16: LCSC C77571 -> C21122
- C17, C18, C19: value 220nF 50V -> 100nF 50V; LCSC C64705 -> C14663
- C23: value 220nF -> 100nF; LCSC C64705 -> C14663
- C4: value 75pF -> 100pF; LCSC C1681 -> C14858
- D3: value STATUS green -> STATUS red; LCSC C12624 -> C2286
- D5: value DIR red -> DIR+ red
- D6: value DIR green -> DIR- red; LCSC C12624 -> C2286
- J4: LCSC C492406 -> (none)
Changed lines of the file:
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@@
     (dnp no)
     (property "Reference" "C4" (at 172.72 26.67 0) (effects (font (size 1.27 1.27))))
-    (property "Value" "75pF" (at 172.72 29.21 0) (effects (font (size 1.27 1.27))))
+    (property "Value" "100pF" (at 172.72 29.21 0) (effects (font (size 1.27 1.27))))
     (property "Footprint" "Capacitor_SMD:C_0603_1608Metric"
       (at 172.72 43.18 0)
       (effects (font (size 1.27 1.27)) hide))
     (property "Datasheet" "~" (at 172.72 43.18 0) (effects (font (size 1.27 1.27)) hide))
-    (property "LCSC" "C1681" (at 172.72 43.18 0) (effects (font (size 1.27 1.27)) hide))
+    (property "LCSC" "C14858" (at 172.72 43.18 0) (effects (font (size 1.27 1.27)) hide))
     (pin "1")
     (pin "2")
@@
     (dnp no)
     (property "Reference" "D3" (at 170.18 118.11 0) (effects (font (size 1.27 1.27))))
-    (property "Value" "STATUS green" (at 170.18 120.65 0) (effects (font (size 1.27 1.27))))
+    (property "Value" "STATUS red" (at 170.18 120.65 0) (effects (font (size 1.27 1.27))))
     (property "Footprint" "LED_SMD:LED_0603_1608Metric"
       (at 167.64 127 0)
       (effects (font (size 1.27 1.27)) hide))
     (property "Datasheet" "~" (at 167.64 127 0) (effects (font (size 1.27 1.27)) hide))
-    (property "LCSC" "C12624" (at 167.64 127 0) (effects (font (size 1.27 1.27)) hide))
+    (property "LCSC" "C2286" (at 167.64 127 0) (effects (font (size 1.27 1.27)) hide))
     (pin "1")
     (pin "2")
@@
       (effects (font (size 1.27 1.27)) hide))
     (property "Datasheet" "~" (at 406.4 139.7 0) (effects (font (size 1.27 1.27)) hide))
-    (property "LCSC" "C77571" (at 406.4 139.7 0) (effects (font (size 1.27 1.27)) hide))
+    (property "LCSC" "C21122" (at 406.4 139.7 0) (effects (font (size 1.27 1.27)) hide))
     (pin "1")
     (pin "2")
@@
     (dnp no)
     (property "Reference" "C17" (at 416.56 118.11 0) (effects (font (size 1.27 1.27))))
-    (property "Value" "220nF 50V" (at 416.56 120.65 0) (effects (font (size 1.27 1.27))))
+    (property "Value" "100nF 50V" (at 416.56 120.65 0) (effects (font (size 1.27 1.27))))
     (property "Footprint" "Capacitor_SMD:C_0603_1608Metric"
       (at 416.56 139.7 0)
       (effects (font (size 1.27 1.27)) hide))
     (property "Datasheet" "~" (at 416.56 139.7 0) (effects (font (size 1.27 1.27)) hide))
-    (property "LCSC" "C64705" (at 416.56 139.7 0) (effects (font (size 1.27 1.27)) hide))
+    (property "LCSC" "C14663" (at 416.56 139.7 0) (effects (font (size 1.27 1.27)) hide))
     (pin "1")
     (pin "2")
@@
     (dnp no)
     (property "Reference" "C18" (at 426.72 118.11 0) (effects (font (size 1.27 1.27))))
-    (property "Value" "220nF 50V" (at 426.72 120.65 0) (effects (font (size 1.27 1.27))))
+    (property "Value" "100nF 50V" (at 426.72 120.65 0) (effects (font (size 1.27 1.27))))
     (property "Footprint" "Capacitor_SMD:C_0603_1608Metric"
       (at 426.72 134.62 0)
       (effects (font (size 1.27 1.27)) hide))
     (property "Datasheet" "~" (at 426.72 134.62 0) (effects (font (size 1.27 1.27)) hide))
-    (property "LCSC" "C64705" (at 426.72 134.62 0) (effects (font (size 1.27 1.27)) hide))
+    (property "LCSC" "C14663" (at 426.72 134.62 0) (effects (font (size 1.27 1.27)) hide))
     (pin "1")
     (pin "2")
@@
     (dnp no)
     (property "Reference" "C19" (at 436.88 118.11 0) (effects (font (size 1.27 1.27))))
-    (property "Value" "220nF 50V" (at 436.88 120.65 0) (effects (font (size 1.27 1.27))))
+    (property "Value" "100nF 50V" (at 436.88 120.65 0) (effects (font (size 1.27 1.27))))
     (property "Footprint" "Capacitor_SMD:C_0603_1608Metric"
       (at 436.88 134.62 0)
       (effects (font (size 1.27 1.27)) hide))
     (property "Datasheet" "~" (at 436.88 134.62 0) (effects (font (size 1.27 1.27)) hide))
-    (property "LCSC" "C64705" (at 436.88 134.62 0) (effects (font (size 1.27 1.27)) hide))
+    (property "LCSC" "C14663" (at 436.88 134.62 0) (effects (font (size 1.27 1.27)) hide))
     (pin "1")
     (pin "2")
@@
     (dnp no)
     (property "Reference" "C23" (at 477.52 118.11 0) (effects (font (size 1.27 1.27))))
-    (property "Value" "220nF" (at 477.52 120.65 0) (effects (font (size 1.27 1.27))))
+    (property "Value" "100nF" (at 477.52 120.65 0) (effects (font (size 1.27 1.27))))
     (property "Footprint" "Capacitor_SMD:C_0603_1608Metric"
       (at 477.52 134.62 0)
       (effects (font (size 1.27 1.27)) hide))
     (property "Datasheet" "~" (at 477.52 134.62 0) (effects (font (size 1.27 1.27)) hide))
-    (property "LCSC" "C64705" (at 477.52 134.62 0) (effects (font (size 1.27 1.27)) hide))
+    (property "LCSC" "C14663" (at 477.52 134.62 0) (effects (font (size 1.27 1.27)) hide))
     (pin "1")
     (pin "2")
@@
     (dnp no)
     (property "Reference" "D5" (at 459.74 171.45 0) (effects (font (size 1.27 1.27))))
-    (property "Value" "DIR red" (at 459.74 173.99 0) (effects (font (size 1.27 1.27))))
+    (property "Value" "DIR+ red" (at 459.74 173.99 0) (effects (font (size 1.27 1.27))))
     (property "Footprint" "LED_SMD:LED_0603_1608Metric"
       (at 459.74 180.34 0)
@@
     (dnp no)
     (property "Reference" "D6" (at 355.6 212.09 0) (effects (font (size 1.27 1.27))))
-    (property "Value" "DIR green" (at 355.6 214.63 0) (effects (font (size 1.27 1.27))))
+    (property "Value" "DIR- red" (at 355.6 214.63 0) (effects (font (size 1.27 1.27))))
     (property "Footprint" "LED_SMD:LED_0603_1608Metric"
       (at 355.6 220.98 0)
       (effects (font (size 1.27 1.27)) hide))
     (property "Datasheet" "~" (at 355.6 220.98 0) (effects (font (size 1.27 1.27)) hide))
-    (property "LCSC" "C12624" (at 355.6 220.98 0) (effects (font (size 1.27 1.27)) hide))
+    (property "LCSC" "C2286" (at 355.6 220.98 0) (effects (font (size 1.27 1.27)) hide))
     (pin "1")
     (pin "2")
@@
       (effects (font (size 1.27 1.27)) hide))
     (property "Datasheet" "~" (at 43.18 276.86 0) (effects (font (size 1.27 1.27)) hide))
-    (property "LCSC" "C492406" (at 43.18 276.86 0) (effects (font (size 1.27 1.27)) hide))
-    (pin "1")
-    (pin "2")
+    (pin "1")
+    (pin "2")

Commit message: LEDs to the left side, C4 back to 75 pF, tidy silkscreen designators
LED column now on the left with facing pads and hand tracks; designators
placed by autopcb tidy_silk(). 0 unrouted, DRC clean; fab regenerated.

Co-Authored-By: Claude Opus 5.5 (1M context) <noreply@anthropic.com>
Claude-Session: https://claude.ai/code/session_01VFhb1Qv7mkaGrgvtw2CS4q
Parts:
- C4: value 100pF -> 75pF; LCSC C14858 -> C1681
Changed lines of the file:
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@@
     (dnp no)
     (property "Reference" "C4" (at 172.72 26.67 0) (effects (font (size 1.27 1.27))))
-    (property "Value" "100pF" (at 172.72 29.21 0) (effects (font (size 1.27 1.27))))
+    (property "Value" "75pF" (at 172.72 29.21 0) (effects (font (size 1.27 1.27))))
     (property "Footprint" "Capacitor_SMD:C_0603_1608Metric"
       (at 172.72 43.18 0)
       (effects (font (size 1.27 1.27)) hide))
     (property "Datasheet" "~" (at 172.72 43.18 0) (effects (font (size 1.27 1.27)) hide))
-    (property "LCSC" "C14858" (at 172.72 43.18 0) (effects (font (size 1.27 1.27)) hide))
+    (property "LCSC" "C1681" (at 172.72 43.18 0) (effects (font (size 1.27 1.27)) hide))
     (pin "1")
     (pin "2")

Commit message: Add STDC14 debug connector for the STLINK-V3MINIE
J6 (Samtec FTSH-107-01-L-DV-K, hand-soldered) on the left under the LEDs:
SWD, NRST, 3V3 sense, GND, and the probe's virtual COM on USART1 (PB6/PB7).
SWD test pads removed. 0 unrouted, DRC clean; fab regenerated.

Co-Authored-By: Claude Opus 5.5 (1M context) <noreply@anthropic.com>
Claude-Session: https://claude.ai/code/session_01VFhb1Qv7mkaGrgvtw2CS4q
Parts:
- removed TP1: +3V3, TestPoint:TestPoint_Pad_D1.0mm, symbol Connector:TestPoint
- removed TP2: SWDIO, TestPoint:TestPoint_Pad_D1.0mm, symbol Connector:TestPoint
- removed TP3: BOOT0_SWCLK, TestPoint:TestPoint_Pad_D1.0mm, symbol Connector:TestPoint
- removed TP4: NRST, TestPoint:TestPoint_Pad_D1.0mm, symbol Connector:TestPoint
- removed TP5: GND, TestPoint:TestPoint_Pad_D1.0mm, symbol Connector:TestPoint
- added J6: STDC14, Connector_PinHeader_1.27mm:PinHeader_2x07_P1.27mm_Vertical_SMD, symbol Connector_Generic:Conn_02x07_Odd_Even
Connections:
- net +3V3: now also J6.3 (Pin_3)
- net BOOT0_SWCLK: now also J6.6 (Pin_6)
- net GND: now also J6.11 (Pin_11), J6.5 (Pin_5), J6.7 (Pin_7)
- net NRST: now also J6.12 (Pin_12)
- net SWDIO: now also J6.4 (Pin_4)
- net VCP_TX: now reaches U1.45 (PB6)
- net VCP_TX: now also J6.14 (Pin_14)
- net VCP_RX: now reaches U1.46 (PB7)
- net VCP_RX: now also J6.13 (Pin_13)
- no-connect marks 30 -> 33
Other:
- moved on the sheet: C16, C17, C18, C19, C20, C21, C22, C23, D4, D5, D6, JP1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
